Commit message: Refine-velodyen_points

File: urdf/sensors/HDL-32E.urdf.xacro (robot description, xacro)
@@ -2,5 +2,5 @@
 <robot xmlns:xacro="http://www.ros.org/wiki/xacro" name="HDL-32E">
   <xacro:property name="M_PI" value="3.1415926535897931" />
-  <xacro:macro name="HDL-32E" params="*origin parent:=base_link name:=velodyne topic:=/velodyne_points hz:=10 lasers:=32 samples:=2187 collision_range:=0.3 min_range:=0.9 max_range:=130.0 noise:=0.008 min_angle:=-${M_PI} max_angle:=${M_PI} gpu:=false">
+  <xacro:macro name="HDL-32E" params="*origin parent:=base_link name:=velodyne topic:=velodyne_points hz:=10 lasers:=32 samples:=2187 collision_range:=0.3 min_range:=0.9 max_range:=130.0 noise:=0.008 min_angle:=-${M_PI} max_angle:=${M_PI} gpu:=false">
     <joint name="${name}_base_mount_joint" type="fixed">
       <xacro:insert_block name="origin" />

Commit message: turn-on-gpu-ray

File: urdf/sensors/HDL-32E.urdf.xacro (robot description, xacro)
@@ -2,5 +2,5 @@
 <robot xmlns:xacro="http://www.ros.org/wiki/xacro" name="HDL-32E">
   <xacro:property name="M_PI" value="3.1415926535897931" />
-  <xacro:macro name="HDL-32E" params="*origin parent:=base_link name:=velodyne topic:=velodyne_points hz:=10 lasers:=32 samples:=2187 collision_range:=0.3 min_range:=0.9 max_range:=130.0 noise:=0.008 min_angle:=-${M_PI} max_angle:=${M_PI} gpu:=false">
+  <xacro:macro name="HDL-32E" params="*origin parent:=base_link name:=velodyne topic:=velodyne_points hz:=10 lasers:=32 samples:=2187 collision_range:=0.3 min_range:=0.9 max_range:=130.0 noise:=0.008 min_angle:=-${M_PI} max_angle:=${M_PI} gpu:=true">
     <joint name="${name}_base_mount_joint" type="fixed">
       <xacro:insert_block name="origin" />
