Commit message: add-realsense

File: robots/kobuki_hexagons_high_velodyne_kinect.urdf.xacro (robot description, xacro)
@@ -15,5 +15,5 @@
   <xacro:stack_hexagons parent="base_link" />
   <xacro:HDL-32E parent="base_link">
-    <origin xyz="0 0 1.0" rpy="0 0 0 "/>
+    <origin xyz="0 0 3.0" rpy="0 0 0 "/>
   </xacro:HDL-32E>
   <xacro:sensor_kinect  parent="base_link"/>
